File: PCB/Sensor/Eagle/sensor_002.sch (EAGLE design)
At the start: 254 parts, among them IC1 LMV324, IC10 LMV324, IC11 LMV324, IC12 LMV324, IC13 LMV324, IC14 LMV324, IC15 LMV324, IC16 LMV324, IC17 LMV324, IC18 LMV324, IC19 LMV324, IC2 LMV324, IC20 LMV324, IC21 LMV324, IC22 LMV324, IC23 LMV324, IC24 LMV324, IC3 LMV324, IC4 LMV324, IC5 LMV324, IC6 LMV324, IC7 LMV324, IC8 LMV324, IC9 LMV324, U1 74HC4067, U2 74HC4067, U3 74HC4067, U4 74HC4067, U5 74HC4067, U6 74HC4067, X1 MKDSN1,5/2-5,08, X2 MKDSN1,5/10-5,08

Commit message: PCB modification, CERN license
Other:
- note added: "Copyright Miroculus 2016. This documentation describes Open Hardware and is licensed under the CERN OHL v. 1.2. You may redistribute and modify this documentation under the terms of the CERN OHL v.1.2. (http://ohwr.org/cernohl). This documentation is distributed WITHOUT ANY EXPRESS OR IMPLIED WARRANTY, INCLUDING OF MERCHANTABILITY, SATISFACTORY QUALITY AND FITNESS FOR A PARTICULAR PURPOSE. Please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"
Changed lines of the file:
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@@
 <text x="488.95" y="-347.98" size="2.54" layer="94" font="vector">AMPLIFIERS 6</text>
 <text x="488.95" y="22.86" size="2.54" layer="94" font="vector">MULTILPLEXORS</text>
+<text x="-99.06" y="27.94" size="1.778" layer="91">Copyright Miroculus 2016.
+This documentation describes Open Hardware and is licensed under the
+CERN OHL v. 1.2.
+You may redistribute and modify this documentation under the terms of the
+CERN OHL v.1.2. (http://ohwr.org/cernohl). This documentation is distributed
+WITHOUT ANY EXPRESS OR IMPLIED WARRANTY, INCLUDING OF
+MERCHANTABILITY, SATISFACTORY QUALITY AND FITNESS FOR A
+PARTICULAR PURPOSE. Please see the CERN OHL v.1.2 for applicable
+conditions</text>
+<text x="165.1" y="27.94" size="1.778" layer="91">Copyright Miroculus 2016.
+This documentation describes Open Hardware and is licensed under the
+CERN OHL v. 1.2.
+You may redistribute and modify this documentation under the terms of the
+CERN OHL v.1.2. (http://ohwr.org/cernohl). This documentation is distributed
+WITHOUT ANY EXPRESS OR IMPLIED WARRANTY, INCLUDING OF
+MERCHANTABILITY, SATISFACTORY QUALITY AND FITNESS FOR A
+PARTICULAR PURPOSE. Please see the CERN OHL v.1.2 for applicable
+conditions</text>
+<text x="345.44" y="12.7" size="1.778" layer="91">Copyright Miroculus 2016.
+This documentation describes Open Hardware and is licensed under the
+CERN OHL v. 1.2.
+You may redistribute and modify this documentation under the terms of the
+CERN OHL v.1.2. (http://ohwr.org/cernohl). This documentation is distributed
+WITHOUT ANY EXPRESS OR IMPLIED WARRANTY, INCLUDING OF
+MERCHANTABILITY, SATISFACTORY QUALITY AND FITNESS FOR A
+PARTICULAR PURPOSE. Please see the CERN OHL v.1.2 for applicable
+conditions</text>
+<text x="-99.06" y="-154.94" size="1.778" layer="91">Copyright Miroculus 2016.
+This documentation describes Open Hardware and is licensed under the
+CERN OHL v. 1.2.
+You may redistribute and modify this documentation under the terms of the
+CERN OHL v.1.2. (http://ohwr.org/cernohl). This documentation is distributed
+WITHOUT ANY EXPRESS OR IMPLIED WARRANTY, INCLUDING OF
+MERCHANTABILITY, SATISFACTORY QUALITY AND FITNESS FOR A
+PARTICULAR PURPOSE. Please see the CERN OHL v.1.2 for applicable
+conditions</text>
+<text x="165.1" y="-154.94" size="1.778" layer="91">Copyright Miroculus 2016.
+This documentation describes Open Hardware and is licensed under the
+CERN OHL v. 1.2.
+You may redistribute and modify this documentation under the terms of the
+CERN OHL v.1.2. (http://ohwr.org/cernohl). This documentation is distributed
+WITHOUT ANY EXPRESS OR IMPLIED WARRANTY, INCLUDING OF
+MERCHANTABILITY, SATISFACTORY QUALITY AND FITNESS FOR A
+PARTICULAR PURPOSE. Please see the CERN OHL v.1.2 for applicable
+conditions</text>
+<text x="434.34" y="-154.94" size="1.778" layer="91">Copyright Miroculus 2016.
+This documentation describes Open Hardware and is licensed under the
+CERN OHL v. 1.2.
+You may redistribute and modify this documentation under the terms of the
+CERN OHL v.1.2. (http://ohwr.org/cernohl). This documentation is distributed
+WITHOUT ANY EXPRESS OR IMPLIED WARRANTY, INCLUDING OF
+MERCHANTABILITY, SATISFACTORY QUALITY AND FITNESS FOR A
+PARTICULAR PURPOSE. Please see the CERN OHL v.1.2 for applicable
+conditions</text>
+<text x="-99.06" y="-340.36" size="1.778" layer="91">Copyright Miroculus 2016.
+This documentation describes Open Hardware and is licensed under the
+CERN OHL v. 1.2.
+You may redistribute and modify this documentation under the terms of the
+CERN OHL v.1.2. (http://ohwr.org/cernohl). This documentation is distributed
+WITHOUT ANY EXPRESS OR IMPLIED WARRANTY, INCLUDING OF
+MERCHANTABILITY, SATISFACTORY QUALITY AND FITNESS FOR A
+PARTICULAR PURPOSE. Please see the CERN OHL v.1.2 for applicable
+conditions</text>
+<text x="165.1" y="-340.36" size="1.778" layer="91">Copyright Miroculus 2016.
+This documentation describes Open Hardware and is licensed under the
+CERN OHL v. 1.2.
+You may redistribute and modify this documentation under the terms of the
+CERN OHL v.1.2. (http://ohwr.org/cernohl). This documentation is distributed
+WITHOUT ANY EXPRESS OR IMPLIED WARRANTY, INCLUDING OF
+MERCHANTABILITY, SATISFACTORY QUALITY AND FITNESS FOR A
+PARTICULAR PURPOSE. Please see the CERN OHL v.1.2 for applicable
+conditions</text>
+<text x="434.34" y="-340.36" size="1.778" layer="91">Copyright Miroculus 2016.
+This documentation describes Open Hardware and is licensed under the
+CERN OHL v. 1.2.
+You may redistribute and modify this documentation under the terms of the
+CERN OHL v.1.2. (http://ohwr.org/cernohl). This documentation is distributed
+WITHOUT ANY EXPRESS OR IMPLIED WARRANTY, INCLUDING OF
+MERCHANTABILITY, SATISFACTORY QUALITY AND FITNESS FOR A
+PARTICULAR PURPOSE. Please see the CERN OHL v.1.2 for applicable
+conditions</text>
 </plain>
 <instances>
