File: PCB/Sensor/Eagle/sensor_003.brd (EAGLE design)
At the start: 142.8 x 97.5 mm, 254 parts, among them IC1 LMV324, IC10 LMV324, IC11 LMV324, IC12 LMV324, IC13 LMV324, IC14 LMV324, IC15 LMV324, IC16 LMV324, IC17 LMV324, IC18 LMV324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

Commit message: few corrections
Routing:
- net GND: track 22.9 -> 28.3 mm, vias 105 -> 111
- net PD58: track 24.7 -> 29.3 mm
- net PD10: track 24.7 -> 28.8 mm
- net PD90: track 24.9 -> 28.2 mm
- net AR3: track 95.1 -> 94.0 mm
- net EO9: track 55.6 -> 56.6 mm
- net AR4: track 71.7 -> 72.6 mm
- net PD74: track 24.7 -> 25.5 mm
- net FO2: track 44.2 -> 44.9 mm
- net PD72: track 6.87 -> 7.41 mm
