File: PCB/Shield/Eagle/shield_007.sch (EAGLE design)
At the start: 48 parts, among them IC1 FDB8880, IC2 FDB8880, IC3 FDB8880, IC4 NCV1117ST50T3GOSCT-ND, IC5 NCV1117ST33T3GOSCT-ND

Commit message: PCB modification, CERN license
Other:
- note added: "Copyright Miroculus 2016. This documentation describes Open Hardware and is licensed under the CERN OHL v. 1.2. You may redistribute and modify this documentation under the terms of the CERN OHL v.1.2. (http://ohwr.org/cernohl). This documentation is distributed WITHOUT ANY EXPRESS OR IMPLIED WARRANTY, INCLUDING OF MERCHANTABILITY, SATISFACTORY QUALITY AND FITNESS FOR A PARTICULAR PURPOSE. Please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"
Changed lines of the file:
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@@
 <text x="152.4" y="27.94" size="1.778" layer="91">LED MOSFET</text>
 <text x="40.64" y="45.72" size="2.54" layer="94">POWER SUPPLY FOR BLT OR WIFI CONNECTOR</text>
+<text x="-101.6" y="27.94" size="1.778" layer="91">Copyright Miroculus 2016.
+This documentation describes Open Hardware and is licensed under the
+CERN OHL v. 1.2.
+You may redistribute and modify this documentation under the terms of the
+CERN OHL v.1.2. (http://ohwr.org/cernohl). This documentation is distributed
+WITHOUT ANY EXPRESS OR IMPLIED WARRANTY, INCLUDING OF
+MERCHANTABILITY, SATISFACTORY QUALITY AND FITNESS FOR A
+PARTICULAR PURPOSE. Please see the CERN OHL v.1.2 for applicable
+conditions</text>
+<text x="172.72" y="27.94" size="1.778" layer="91">Copyright Miroculus 2016.
+This documentation describes Open Hardware and is licensed under the
+CERN OHL v. 1.2.
+You may redistribute and modify this documentation under the terms of the
+CERN OHL v.1.2. (http://ohwr.org/cernohl). This documentation is distributed
+WITHOUT ANY EXPRESS OR IMPLIED WARRANTY, INCLUDING OF
+MERCHANTABILITY, SATISFACTORY QUALITY AND FITNESS FOR A
+PARTICULAR PURPOSE. Please see the CERN OHL v.1.2 for applicable
+conditions</text>
 </plain>
 <instances>
